File: Synapse.sch (KiCad schematic (older format))
At the start: 7 parts, among them U2 WeAct_BlackPill_Short

Commit message: PAUSED: Use `git resume` to continue working.
Parts:
- added C1: 100pF ceramic, 100v, 10%, Capacitor_SMD:C_0805_2012Metric, symbol Device:C
- added FB1: Ferrite_Bead_Small, Inductor_SMD:L_0805_2012Metric, symbol Device:Ferrite_Bead_Small
- added Q1: Q_PMOS_GSD, -3.6A 0.02R, Package_TO_SOT_SMD:SOT-23, symbol Device:Q_PMOS_GSD
- added Q2: Q_NMOS_GSD 1Amp, Package_TO_SOT_SMD:SOT-23, symbol Device:Q_NMOS_GSD
- added R5, R6: 10k. 125mW. 5%., Resistor_SMD:R_0805_2012Metric, symbol Device:R
- R1, R2: footprint Resistor_SMD:R_1206_3216Metric -> Resistor_SMD:R_0805_2012Metric; LCSC C17950 -> C17530
- R3, R4: footprint Resistor_SMD:R_1206_3216Metric -> Resistor_SMD:R_0805_2012Metric; LCSC C17954 -> C17539
Connections:
- net labels added: +5V, GNDREF, side-power, side-switch
- wire segments 18 -> 31
Changed lines of the file:
@@
 F 0 "R1" H 6020 3796 50  0000 L CNN
 F 1 "2.7K" H 6020 3705 50  0000 L CNN
-F 2 "Resistor_SMD:R_1206_3216Metric" V 5880 3750 50  0001 C CNN
+F 2 "Resistor_SMD:R_0805_2012Metric" V 5880 3750 50  0001 C CNN
 F 3 "~" H 5950 3750 50  0001 C CNN
-F 4 "C17950" H 5950 3750 50  0001 C CNN "LCSC"
+F 4 "C17530" H 5950 3750 50  0001 C CNN "LCSC"
 	1    5950 3750
 	1    0    0    -1
@@
 Wire Wire Line
 	2700 3100 3000 3100
-Text Label 5750 2150 2    50   ~ 0
-gnd
-Text Label 5750 2050 2    50   ~ 0
-vbus
 Text Label 5250 2100 0    50   ~ 0
 sda
@@
 sda
 Text Label 5250 1600 0    50   ~ 0
-vbus
+side-power
 Text Label 5950 3900 3    50   ~ 0
 scl
 Text Label 5750 1650 2    50   ~ 0
 scl
-Text Label 4750 3100 0    50   ~ 0
-gnd
 Wire Wire Line
 	4650 3100 4750 3100
-Text Label 3100 3100 0    50   ~ 0
-gnd
 Wire Wire Line
 	3000 3100 3100 3100
@@
 scl
 Text Label 3600 1600 0    50   ~ 0
-vbus
+side-power
 $Comp
 L Connector:USB_C_Receptacle_USB2.0 USB2
@@
 F 0 "R4" H 3970 3896 50  0000 L CNN
 F 1 "200k" H 3970 3805 50  0000 L CNN
-F 2 "Resistor_SMD:R_1206_3216Metric" V 3830 3850 50  0001 C CNN
+F 2 "Resistor_SMD:R_0805_2012Metric" V 3830 3850 50  0001 C CNN
 F 3 "~" H 3900 3850 50  0001 C CNN
-F 4 "C17954" H 3900 3850 50  0001 C CNN "LCSC"
+F 4 "C17539" H 3900 3850 50  0001 C CNN "LCSC"
 	1    3900 3850
 	1    0    0    -1
@@
 F 0 "R2" H 5570 3796 50  0000 L CNN
 F 1 "2.7K" H 5570 3705 50  0000 L CNN
-F 2 "Resistor_SMD:R_1206_3216Metric" V 5430 3750 50  0001 C CNN
+F 2 "Resistor_SMD:R_0805_2012Metric" V 5430 3750 50  0001 C CNN
 F 3 "~" H 5500 3750 50  0001 C CNN
-F 4 "C17950" H 5500 3750 50  0001 C CNN "LCSC"
+F 4 "C17530" H 5500 3750 50  0001 C CNN "LCSC"
 	1    5500 3750
 	1    0    0    -1
@@
 F 0 "R3" H 3620 3896 50  0000 L CNN
 F 1 "200k" H 3620 3805 50  0000 L CNN
-F 2 "Resistor_SMD:R_1206_3216Metric" V 3480 3850 50  0001 C CNN
+F 2 "Resistor_SMD:R_0805_2012Metric" V 3480 3850 50  0001 C CNN
 F 3 "~" H 3550 3850 50  0001 C CNN
-F 4 "C17954" H 3550 3850 50  0001 C CNN "LCSC"
+F 4 "C17539" H 3550 3850 50  0001 C CNN "LCSC"
 	1    3550 3850
 	1    0    0    -1
@@
 	1    0    0    -1
 $EndComp
+$Comp
+L Device:Q_NMOS_GSD Q2
+U 1 1 60F1EB6F
+P 8050 4050
+F 0 "Q2" H 8255 4096 50  0000 L CNN
+F 1 "Q_NMOS_GSD 1Amp" H 8255 4005 50  0000 L CNN
+F 2 "Package_TO_SOT_SMD:SOT-23" H 8250 4150 50  0001 C CNN
+F 3 "~" H 8050 4050 50  0001 C CNN
+F 4 "C20917" H 8050 4050 50  0001 C CNN "LCSC"
+	1    8050 4050
+	-1   0    0    -1
+$EndComp
+$Comp
+L Device:Q_PMOS_GSD Q1
+U 1 1 60F1FCC9
+P 7950 3400
+F 0 "Q1" V 8292 3400 50  0000 C CNN
+F 1 "Q_PMOS_GSD, -3.6A 0.02R" V 8201 3400 50  0000 C CNN
+F 2 "Package_TO_SOT_SMD:SOT-23" H 8150 3500 50  0001 C CNN
+F 3 "~" H 7950 3400 50  0001 C CNN
+F 4 "C15127" V 7950 3400 50  0001 C CNN "LCSC"
+	1    7950 3400
+	0    -1   -1   0
+$EndComp
+$Comp
+L Device:R R5
+U 1 1 60F21C7A
+P 8600 4200
+F 0 "R5" H 8670 4246 50  0000 L CNN
+F 1 "10k. 125mW. 5%." H 8670 4155 50  0000 L CNN
+F 2 "Resistor_SMD:R_0805_2012Metric" V 8530 4200 50  0001 C CNN
+F 3 "~" H 8600 4200 50  0001 C CNN
+F 4 "C17414" H 8600 4200 50  0001 C CNN "LCSC"
+	1    8600 4200
+	1    0    0    -1
+$EndComp
+$Comp
+L Device:R R6
+U 1 1 60F228A3
+P 8600 3450
+F 0 "R6" H 8670 3496 50  0000 L CNN
+F 1 "10k. 125mW. 5%." H 8670 3405 50  0000 L CNN
+F 2 "Resistor_SMD:R_0805_2012Metric" V 8530 3450 50  0001 C CNN
+F 3 "~" H 8600 3450 50  0001 C CNN
+F 4 "C17414" H 8600 3450 50  0001 C CNN "LCSC"
+	1    8600 3450
+	1    0    0    -1
+$EndComp
+$Comp
+L Device:C C1
+U 1 1 60F23AD2
+P 7100 3150
+F 0 "C1" H 7215 3196 50  0000 L CNN
+F 1 "100pF ceramic, 100v, 10%" H 7215 3105 50  0000 L CNN
+F 2 "Capacitor_SMD:C_0805_2012Metric" H 7138 3000 50  0001 C CNN
+F 3 "~" H 7100 3150 50  0001 C CNN
+F 4 "C159771" H 7100 3150 50  0001 C CNN "LCSC"
+	1    7100 3150
+	1    0    0    -1
+$EndComp
+$Comp
+L Device:Ferrite_Bead_Small FB1
+U 1 1 60F24091
+P 7100 3650
+F 0 "FB1" H 7200 3696 50  0000 L CNN
+F 1 "Ferrite_Bead_Small" H 7200 3605 50  0000 L CNN
+F 2 "Inductor_SMD:L_0805_2012Metric" V 7030 3650 50  0001 C CNN
+F 3 "~" H 7100 3650 50  0001 C CNN
+F 4 "C1017" H 7100 3650 50  0001 C CNN "LCSC"
+	1    7100 3650
+	1    0    0    -1
+$EndComp
+$Comp
+L power:+5V #PWR0101
+U 1 1 60F258CA
+P 9000 3300
+F 0 "#PWR0101" H 9000 3150 50  0001 C CNN
+F 1 "+5V" H 9015 3473 50  0000 C CNN
+F 2 "" H 9000 3300 50  0001 C CNN
+F 3 "" H 9000 3300 50  0001 C CNN
+	1    9000 3300
+	1    0    0    -1
+$EndComp
+$Comp
+L power:GNDREF #PWR0102
+U 1 1 60F265C4
+P 8600 4350
+F 0 "#PWR0102" H 8600 4100 50  0001 C CNN
+F 1 "GNDREF" H 8605 4177 50  0001 C CNN
+F 2 "" H 8600 4350 50  0001 C CNN
+F 3 "" H 8600 4350 50  0001 C CNN
+	1    8600 4350
+	1    0    0    -1
+$EndComp
+$Comp
+L power:GNDREF #PWR0103
+U 1 1 60F2692F
+P 7950 4350
+F 0 "#PWR0103" H 7950 4100 50  0001 C CNN
+F 1 "GNDREF" H 7955 4177 50  0001 C CNN
+F 2 "" H 7950 4350 50  0001 C CNN
+F 3 "" H 7950 4350 50  0001 C CNN
+	1    7950 4350
+	1    0    0    -1
+$EndComp
+$Comp
+L power:GNDREF #PWR0104
+U 1 1 60F26CAC
+P 7100 3000
+F 0 "#PWR0104" H 7100 2750 50  0001 C CNN
+F 1 "GNDREF" H 7105 2827 50  0001 C CNN
+F 2 "" H 7100 3000 50  0001 C CNN
+F 3 "" H 7100 3000 50  0001 C CNN
+	1    7100 3000
+	-1   0    0    1
+$EndComp
+Wire Wire Line
+	9000 3300 8600 3300
+Wire Wire Line
+	8150 3300 8600 3300
+Connection ~ 8600 3300
+Wire Wire Line
+	7750 3300 7100 3300
+Wire Wire Line
+	7100 3300 7100 3550
+Connection ~ 7100 3300
+Wire Wire Line
+	7950 3600 7950 3700
+Wire Wire Line
+	7950 3700 8600 3700
+Wire Wire Line
+	8600 3700 8600 3600
+Connection ~ 7950 3700
+Wire Wire Line
+	7950 3700 7950 3850
+Wire Wire Line
+	7950 4350 7950 4250
+Wire Wire Line
+	8600 4050 8250 4050
+Text Label 8400 4050 0    50   ~ 0
+side-switch
+Text Label 6900 3850 2    50   ~ 0
+side-power
+Wire Wire Line
+	6900 3850 7100 3850
+Wire Wire Line
+	7100 3850 7100 3750
+$Comp
+L power:GNDREF #PWR0105
+U 1 1 60F2B3EC
+P 5650 2150
+F 0 "#PWR0105" H 5650 1900 50  0001 C CNN
+F 1 "GNDREF" H 5655 1977 50  0001 C CNN
+F 2 "" H 5650 2150 50  0001 C CNN
+F 3 "" H 5650 2150 50  0001 C CNN
+	1    5650 2150
+	1    0    0    -1
+$EndComp
+$Comp
+L power:+5V #PWR0106
+U 1 1 60F2DDB3
+P 5650 2050
+F 0 "#PWR0106" H 5650 1900 50  0001 C CNN
+F 1 "+5V" H 5665 2223 50  0000 C CNN
+F 2 "" H 5650 2050 50  0001 C CNN
+F 3 "" H 5650 2050 50  0001 C CNN
+	1    5650 2050
+	1    0    0    -1
+$EndComp
+Wire Wire Line
+	5800 2150 5790 2150
+Connection ~ 5790 2150
+Wire Wire Line
+	5790 2150 5650 2150
+Wire Wire Line
+	5650 2050 5790 2050
+Connection ~ 5790 2050
+Wire Wire Line
+	5790 2050 5800 2050
+$Comp
+L power:GNDREF #PWR0107
+U 1 1 60F30306
+P 3100 3100
+F 0 "#PWR0107" H 3100 2850 50  0001 C CNN
+F 1 "GNDREF" H 3105 2927 50  0001 C CNN
+F 2 "" H 3100 3100 50  0001 C CNN
+F 3 "" H 3100 3100 50  0001 C CNN
+	1    3100 3100
+	1    0    0    -1
+$EndComp
+$Comp
+L power:GNDREF #PWR0108
+U 1 1 60F30A69
+P 4750 3100
+F 0 "#PWR0108" H 4750 2850 50  0001 C CNN
+F 1 "GNDREF" H 4755 2927 50  0001 C CNN
+F 2 "" H 4750 3100 50  0001 C CNN
+F 3 "" H 4750 3100 50  0001 C CNN
+	1    4750 3100
+	1    0    0    -1
+$EndComp
+Text Label 7650 2050 0    50   ~ 0
+side-switch
 Wire Wire Line
 	5800 1650 5790 1650
@@
 	5790 1750 5750 1750
 Wire Wire Line
-	5800 2050 5790 2050
-Connection ~ 5790 2050
-Wire Wire Line
-	5790 2050 5750 2050
-Wire Wire Line
-	5800 2150 5790 2150
-Connection ~ 5790 2150
-Wire Wire Line
-	5790 2150 5750 2150
+	7600 2050 7650 2050
 $EndSCHEMATC
